File: PoweredUSB-Adapter.kicad_sch (KiCad schematic)
At the start: 12 parts, among them CN1 PoweredUSB 12V, CN4 USB-C-USB2.0-16P, J1 12V 5,5/2,5(2,1), J2 USB-HDR, J3 JST2.5-2P

Commit message: initial release.
Parts:
- CN1: PN (none) -> AMP:55917-500LF
- CN4: PN (none) -> GCT:USB4105-GF-A-120
- D1: PN (none) -> DIO:LL4148
- J1: PN (none) -> GCT:DCJ200-10-A-K1-K
Changed lines of the file:
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@@
       (effects (font (size 1.27 1.27)) hide)
     )
-    (property "PN" "" (at 115.57 34.29 0)
+    (property "PN" "GCT:DCJ200-10-A-K1-K" (at 123.19 41.91 0)
       (effects (font (size 1.27 1.27)))
     )
@@
       (effects (font (size 1.27 1.27)) hide)
     )
-    (property "PN" "" (at 110.49 111.76 0)
+    (property "PN" "GCT:USB4105-GF-A-120" (at 142.875 137.16 0)
       (effects (font (size 1.27 1.27)))
     )
@@
   (symbol (lib_id "my-active:D") (at 50.8 59.69 270) (unit 1)
     (in_bom yes) (on_board yes) (dnp no)
-    (property "Reference" "D1" (at 53.975 59.055 0)
+    (property "Reference" "D1" (at 48.895 58.42 0)
       (effects (font (size 1.27 1.27)) (justify left))
     )
@@
       (effects (font (size 1.27 1.27)) hide)
     )
-    (property "PN" "" (at 50.8 59.69 0)
-      (effects (font (size 1.27 1.27)))
+    (property "PN" "DIO:LL4148" (at 53.975 60.96 0)
+      (effects (font (size 0.762 0.762)))
     )
     (pin "1")
@@
       (effects (font (size 1.27 1.27)) hide)
     )
-    (property "PN" "" (at 41.91 67.31 0)
+    (property "PN" "AMP:55917-500LF" (at 35.56 86.995 0)
       (effects (font (size 1.27 1.27)))
     )
